File: electrical/stepper_multi_axis/Power.sch (KiCad schematic (older format))
At the start: 6 parts, among them J10 Conn_01x02_Male, U1 LM2576S-5

Commit message: shipped things
Parts:
- removed D1: 1N5822, Diode_THT:D_DO-201AD_P15.24mm_Horizontal, symbol Diode:1N5822
- added D1: D_Schottky, Diode_SMD:D_SOD-128, symbol Device:D_Schottky
- C10: Digi-Key_PN (none) -> 399-20518-1-ND
- C9: Digi-Key_PN (none) -> 10-EEE-FK1H101GLCT-ND
- L1: Digi-Key_PN (none) -> 308-1331-1-ND; LCSC (none) -> C169378
- U1: Digi-Key_PN (none) -> LM2576S-5.0/NOPB-ND; LCSC (none) -> C347413
Connections:
- net GND: now also D1.2 (A)
- net at L1.1, U1.2 (OUT): now also D1.1 (K)
Changed lines of the file:
@@
 $Descr A4 11693 8268
 encoding utf-8
-Sheet 3 8
+Sheet 3 10
 Title ""
 Date ""
@@
 F 2 "Package_TO_SOT_SMD:TO-263-5_TabPin3" H 6950 2850 50  0001 L CIN
 F 3 "http://www.ti.com/lit/ds/symlink/lm2576.pdf" H 6950 3100 50  0001 C CNN
+F 4 "LM2576S-5.0/NOPB-ND" H 6950 3100 50  0001 C CNN "Digi-Key_PN"
+F 5 "C347413" H 6950 3100 50  0001 C CNN "LCSC"
 	1    6950 3100
 	1    0    0    -1
@@
 F 2 "Capacitor_SMD:CP_Elec_10x12.5" H 6200 3150 50  0001 C CNN
 F 3 "~" H 6200 3150 50  0001 C CNN
+F 4 "10-EEE-FK1H101GLCT-ND" H 6200 3150 50  0001 C CNN "Digi-Key_PN"
 	1    6200 3150
 	1    0    0    -1
@@
 F 2 "Capacitor_SMD:CP_Elec_10x12.5" H 8500 3350 50  0001 C CNN
 F 3 "~" H 8500 3350 50  0001 C CNN
+F 4 "399-20518-1-ND" H 8500 3350 50  0001 C CNN "Digi-Key_PN"
 	1    8500 3350
 	1    0    0    -1
@@
 	6200 3300 6200 3500
 $Comp
-L Diode:1N5822 D1
-U 1 1 60A7C2BE
-P 7650 3350
-F 0 "D1" V 7604 3430 50  0000 L CNN
-F 1 "1N5822" V 7695 3430 50  0000 L CNN
-F 2 "Diode_THT:D_DO-201AD_P15.24mm_Horizontal" H 7650 3175 50  0001 C CNN
-F 3 "http://www.vishay.com/docs/88526/1n5820.pdf" H 7650 3350 50  0001 C CNN
-	1    7650 3350
-	0    1    1    0
-$EndComp
-Wire Wire Line
-	7450 3200 7650 3200
-Wire Wire Line
-	7650 3200 7950 3200
-Connection ~ 7650 3200
-$Comp
-L power:GND #PWR0140
-U 1 1 60A7D7A4
-P 7650 3500
-F 0 "#PWR0140" H 7650 3250 50  0001 C CNN
-F 1 "GND" H 7655 3327 50  0000 C CNN
-F 2 "" H 7650 3500 50  0001 C CNN
-F 3 "" H 7650 3500 50  0001 C CNN
-	1    7650 3500
-	1    0    0    -1
-$EndComp
-$Comp
 L power:GND #PWR0141
 U 1 1 60A7DA82
@@
 F 2 "Inductor_SMD:L_12x12mm_H8mm" H 8200 3200 50  0001 C CNN
 F 3 "~" H 8200 3200 50  0001 C CNN
+F 4 "308-1331-1-ND" H 8200 3200 50  0001 C CNN "Digi-Key_PN"
+F 5 "C169378" H 8200 3200 50  0001 C CNN "LCSC"
 	1    8200 3200
 	1    0    0    -1
@@
 	-1   0    0    -1
 $EndComp
+$Comp
+L Device:D_Schottky D?
+U 1 1 612E2960
+P 7650 3350
+AR Path="/5515D395/612E2960" Ref="D?"  Part="1"
+AR Path="/60A6FF98/612E2960" Ref="D1"  Part="1"
+F 0 "D1" H 7650 3567 50  0000 C CNN
+F 1 "D_Schottky" H 7650 3476 50  0000 C CNN
+F 2 "Diode_SMD:D_SOD-128" H 7650 3350 50  0001 C CNN
+F 3 "~" H 7650 3350 50  0001 C CNN
+F 4 "1727-7810-1-ND" H 7650 3350 50  0001 C CNN "Digi-Key_PN"
+F 5 "C456127" H 7650 3350 50  0001 C CNN "LCSC"
+	1    7650 3350
+	0    1    1    0
+$EndComp
+$Comp
+L power:GND #PWR0140
+U 1 1 60A7D7A4
+P 7650 3500
+F 0 "#PWR0140" H 7650 3250 50  0001 C CNN
+F 1 "GND" H 7655 3327 50  0000 C CNN
+F 2 "" H 7650 3500 50  0001 C CNN
+F 3 "" H 7650 3500 50  0001 C CNN
+	1    7650 3500
+	1    0    0    -1
+$EndComp
+Wire Wire Line
+	7450 3200 7650 3200
+Connection ~ 7650 3200
+Wire Wire Line
+	7650 3200 7950 3200
 $EndSCHEMATC
