File: electrical/stepper_multi_axis/Servo_Driver.sch (KiCad schematic (older format))
At the start: 5 parts, among them J19 Conn_01x05_Male, J20 Conn_01x04_Male, U11 TMC5160-BOB

Commit message: shipped things
Parts:
- C11: Digi-Key_PN (none) -> PCE4976CT-ND
- J19: Digi-Key_PN (none) -> WM22670-ND
- J20: Digi-Key_PN (none) -> WM22669-ND
- RN1: Digi-Key_PN (none) -> 742C083102JPCT-ND; LCSC (none) -> C20197
Changed lines of the file:
@@
 $Descr A4 11693 8268
 encoding utf-8
-Sheet 8 8
+Sheet 8 10
 Title ""
 Date ""
@@
 F 2 "sl_connector:1719740104" H 6550 3700 50  0001 C CNN
 F 3 "~" H 6550 3700 50  0001 C CNN
+F 4 "WM22669-ND" H 6550 3700 50  0001 C CNN "Digi-Key_PN"
 	1    6550 3700
 	-1   0    0    1
@@
 F 2 "Capacitor_SMD:CP_Elec_8x6.7" H 6325 2900 50  0001 C CNN
 F 3 "~" H 6325 2900 50  0001 C CNN
+F 4 "PCE4976CT-ND" H 6325 2900 50  0001 C CNN "Digi-Key_PN"
 	1    6325 2900
 	1    0    0    -1
@@
 F 2 "sl_connector:1719740105" H 6525 2025 50  0001 C CNN
 F 3 "~" H 6525 2025 50  0001 C CNN
+F 4 "WM22670-ND" H 6525 2025 50  0001 C CNN "Digi-Key_PN"
 	1    6525 2025
 	-1   0    0    -1
@@
 F 2 "Resistor_SMD:R_Array_Concave_4x0603" V 5675 2225 50  0001 C CNN
 F 3 "~" H 5400 2225 50  0001 C CNN
+F 4 "742C083102JPCT-ND" V 5400 2225 50  0001 C CNN "Digi-Key_PN"
+F 5 "C20197" V 5400 2225 50  0001 C CNN "LCSC"
 	1    5400 2225
 	0    1    1    0
