File: electrical/stepper_multi_axis/USBHub.sch (KiCad schematic (older format))
At the start: 8 parts, among them J13 USB_B_Micro, J21 Conn_01x01, J32 USB_A, U12 FSUSB42MUX

Commit message: pre delete thru hole
Parts:
- added C14, C15, C19: 100nF, Capacitor_SMD:C_0603_1608Metric_Pad1.08x0.95mm_HandSolder, symbol Device:C_Small
- added C16, C17, C18: 10uF, Capacitor_SMD:C_0603_1608Metric_Pad1.08x0.95mm_HandSolder, symbol Device:C_Small
- added J33, J34: USB_A, Connector_USB:USB_A_Molex_67643_Horizontal, symbol Connector:USB_A
- added J39: USB_B_Micro, Connector_USB:USB_Micro-B_Molex-105017-0001, symbol Connector:USB_B_Micro
- added R10: 2.7k, Resistor_SMD:R_0603_1608Metric_Pad0.98x0.95mm_HandSolder, symbol Device:R_Small_US
- added R11, R12: 2.2k, Resistor_SMD:R_0603_1608Metric_Pad0.98x0.95mm_HandSolder, symbol Device:R_Small_US
- added U13: FE1.1s, Package_SO:SSOP-28_3.9x9.9mm_P0.635mm, symbol Interface_USB:FE1.1s
- added U14: FSUSB42MUX, usbmux:SOP50P490X110-10N, symbol FSUSB42MUX:FSUSB42MUX
- added Y1: Crystal, Crystal:Crystal_HC50_Vertical, symbol Device:Crystal
Connections:
- net +3.3VA: now also C19.1, U13.18 (VBUSM), U14.1 (VCC)
- net +5V: now also C14.1, C15.1, C16.2, J33.1 (VBUS), J34.1 (VBUS), U13.20 (VDD5)
- net GND: now also C14.2, C15.2, C16.1, C17.1, C18.1, C19.2, J33.4 (GND), J33.5 (Shield), J34.4 (GND), J34.5 (Shield), J39.5 (GND), J39.6 (Shield), R10.2, R12.2, U13.1 (VSS), U14.10 (~OE), U14.5 (GND)
- net USB_A+: now also U13.16 (DPU); no longer J32.3 (D+)
- net USB_A-: now also U13.15 (DMU); no longer J32.2 (D-)
- new net: C18.2, U13.12 (VD18_O), U13.28 (VD18)
- new net: C17.2, U13.13 (VD33), U13.17 (~XRSTJ), U13.19 (BUSJ), U13.21 (VD33_O), U13.26 (OVCJ)
- new net: R10.1, U13.14 (REXT)
- new net: U13.2 (XOUT), Y1.2
- new net: U13.3 (XIN), Y1.1
- new net: R11.2, R12.1, U14.2 (SEL)
- new net: J39.1 (VBUS), R11.1
- new net 1+: J32.3 (D+), U13.11 (DP1)
- new net 1-: J32.2 (D-), U13.10 (DM1)
- new net 2+: J33.3 (D+), U13.9 (DP2)
- new net 2-: J33.2 (D-), U13.8 (DM2)
- new net 3+: J34.3 (D+), U13.7 (DP3)
- new net 3-: J34.2 (D-), U13.6 (DM3)
- new net INT+: U13.5 (DP4), U14.7 (HSD1+)
- new net INT-: U13.4 (DM4), U14.6 (HSD1-)
- new net OVERRIDE+: J39.3 (D+), U14.9 (HSD2+)
- new net OVERRIDE-: J39.2 (D-), U14.8 (HSD2-)
- new net USB_INTERNAL_N: U14.4 (D-)
- new net USB_INTERNAL_P: U14.3 (D+)
- no-connect marks 0 -> 5
Other:
- moved on the sheet: C12, C13, J13, J2, J32, R8, R9, U12
