File: electrical/stepper_multi_axis/RPi_GPIO.sch (KiCad schematic (older format))
At the start: 9 parts, among them J2 RPi_GPIO, U10 Teensy4.1

Commit message: added higher current drivers
Parts:
- removed R10, R8, R9: 100, Resistor_SMD:R_0603_1608Metric_Pad0.98x0.95mm_HandSolder, symbol Device:R_Small_US
- added RN3: R_100_4, Resistor_SMD:R_Array_Concave_4x0603, symbol Device:R_Pack04
Connections:
- net labels added: A_ENCA, A_ENCB, B_ENCA, B_ENCB, CS4
- net labels removed: A_LIMIT, B_LIMIT, COOLANT_FLOOD
- wire segments 64 -> 66
Changed lines of the file:
@@
 $Descr A4 11693 8268
 encoding utf-8
-Sheet 7 7
+Sheet 4 8
 Title ""
 Date ""
@@
 Z_LIMIT
 Text HLabel 9400 2650 2    50   Input ~ 0
-A_LIMIT
+A_ENCA
 Wire Wire Line
 	9400 2650 9250 2650
@@
 Text HLabel 9400 4150 2    50   Output ~ 0
 A_ENABLE
-Text HLabel 9400 4250 2    50   Output ~ 0
+Text HLabel 9400 3850 2    50   Output ~ 0
 B_ENABLE
 Wire Wire Line
@@
 	9250 4150 9400 4150
 Wire Wire Line
-	9400 4250 9250 4250
+	9400 3850 9250 3850
 Text HLabel 6700 4250 0    50   Input ~ 0
-B_LIMIT
+B_ENCA
 Wire Wire Line
 	6700 4250 7050 4250
@@
 Wire Wire Line
 	7050 4350 6700 4350
-Text HLabel 9400 3050 2    50   Output ~ 0
-COOLANT_FLOOD
+Text HLabel 9400 3050 2    50   Input ~ 0
+A_ENCB
 Text HLabel 9400 3150 2    50   Output ~ 0
 COOLANT_MIST
@@
 Wire Wire Line
 	5250 2550 7050 2550
-Text HLabel 9700 4550 2    50   Output ~ 0
+Text HLabel 9900 4550 2    50   Output ~ 0
 CS0
 Text HLabel 9700 4650 2    50   Output ~ 0
 CS1
 Wire Wire Line
-	9450 4550 9700 4550
-Wire Wire Line
-	9450 4650 9700 4650
+	9650 4550 9900 4550
 Wire Wire Line
 	3350 3250 3050 3250
@@
 Wire Wire Line
 	3350 3050 3050 3050
-Text HLabel 9750 4450 2    50   Output ~ 0
+Text HLabel 9950 4450 2    50   Output ~ 0
 CS2
-Text HLabel 9750 4350 2    50   Output ~ 0
+Text HLabel 9950 4350 2    50   Output ~ 0
 CS3
 Wire Wire Line
-	9450 4450 9750 4450
-Wire Wire Line
-	9750 4350 9450 4350
+	9650 4450 9950 4450
+Wire Wire Line
+	9950 4350 9650 4350
 Text Label 5550 2950 0    50   ~ 0
 SWDIO
@@
 	0    -1   -1   0
 $EndComp
-$Comp
-L Device:R_Small_US R?
-U 1 1 6108AB49
-P 9350 4350
-AR Path="/60869CEA/6108AB49" Ref="R?"  Part="1"
-AR Path="/608DFF6C/6108AB49" Ref="R?"  Part="1"
-AR Path="/608FE26D/6108AB49" Ref="R?"  Part="1"
-AR Path="/608FE277/6108AB49" Ref="R?"  Part="1"
-AR Path="/5515D395/6108AB49" Ref="R8"  Part="1"
-F 0 "R8" H 9418 4396 50  0000 L CNN
-F 1 "100" H 9418 4305 50  0000 L CNN
-F 2 "Resistor_SMD:R_0603_1608Metric_Pad0.98x0.95mm_HandSolder" H 9350 4350 50  0001 C CNN
-F 3 "~" H 9350 4350 50  0001 C CNN
-	1    9350 4350
-	0    -1   -1   0
-$EndComp
-$Comp
-L Device:R_Small_US R?
-U 1 1 6108C4B0
-P 9350 4450
-AR Path="/60869CEA/6108C4B0" Ref="R?"  Part="1"
-AR Path="/608DFF6C/6108C4B0" Ref="R?"  Part="1"
-AR Path="/608FE26D/6108C4B0" Ref="R?"  Part="1"
-AR Path="/608FE277/6108C4B0" Ref="R?"  Part="1"
-AR Path="/5515D395/6108C4B0" Ref="R9"  Part="1"
-F 0 "R9" H 9418 4496 50  0000 L CNN
-F 1 "100" H 9418 4405 50  0000 L CNN
-F 2 "Resistor_SMD:R_0603_1608Metric_Pad0.98x0.95mm_HandSolder" H 9350 4450 50  0001 C CNN
-F 3 "~" H 9350 4450 50  0001 C CNN
-	1    9350 4450
-	0    -1   -1   0
-$EndComp
-$Comp
-L Device:R_Small_US R?
-U 1 1 6108DDAE
-P 9350 4550
-AR Path="/60869CEA/6108DDAE" Ref="R?"  Part="1"
-AR Path="/608DFF6C/6108DDAE" Ref="R?"  Part="1"
-AR Path="/608FE26D/6108DDAE" Ref="R?"  Part="1"
-AR Path="/608FE277/6108DDAE" Ref="R?"  Part="1"
-AR Path="/5515D395/6108DDAE" Ref="R10"  Part="1"
-F 0 "R10" H 9418 4596 50  0000 L CNN
-F 1 "100" H 9418 4505 50  0000 L CNN
-F 2 "Resistor_SMD:R_0603_1608Metric_Pad0.98x0.95mm_HandSolder" H 9350 4550 50  0001 C CNN
-F 3 "~" H 9350 4550 50  0001 C CNN
-	1    9350 4550
-	0    -1   -1   0
-$EndComp
+Text HLabel 9950 4250 2    50   Output ~ 0
+CS4
+Wire Wire Line
+	9650 4250 9950 4250
+Text HLabel 6700 4450 0    50   Input ~ 0
+B_ENCB
+Wire Wire Line
+	6700 4450 7050 4450
+$Comp
+L Device:R_Pack04 RN3
+U 1 1 613D08E2
+P 9450 4350
+F 0 "RN3" V 9775 4350 50  0000 C CNN
+F 1 "R_100_4" V 9684 4350 50  0000 C CNN
+F 2 "Resistor_SMD:R_Array_Concave_4x0603" V 9725 4350 50  0001 C CNN
+F 3 "~" H 9450 4350 50  0001 C CNN
+	1    9450 4350
+	0    1    -1   0
+$EndComp
+Wire Wire Line
+	9450 4650 9700 4650
 $EndSCHEMATC

Commit message: shipped things
Parts:
- removed J2: RPi_GPIO, RPi_Hat:Pin_Header_Straight_2x20, symbol RPi_Hat:RPi_GPIO
- D26: Digi-Key_PN (none) -> 1727-7810-1-ND; LCSC (none) -> C456127
- R5, R6, R7: LCSC (none) -> C105588
- RN3: Digi-Key_PN (none) -> 742C083101JPCT-ND; LCSC (none) -> C79203
Connections:
- net labels removed: PI_RX, PI_TX, SCLK, SWDIO
- wire segments 66 -> 41
Changed lines of the file:
@@
 $Descr A4 11693 8268
 encoding utf-8
-Sheet 4 8
+Sheet 4 10
 Title ""
 Date ""
@@
 $EndDescr
 $Comp
-L RPi_Hat:RPi_GPIO J2
-U 1 1 5516AE26
-P 3550 2150
-AR Path="/5516AE26" Ref="J2"  Part="1"
-AR Path="/5515D395/5516AE26" Ref="J2"  Part="1"
-F 0 "J2" H 4300 2400 60  0000 C CNN
-F 1 "RPi_GPIO" H 4300 2300 60  0000 C CNN
-F 2 "RPi_Hat:Pin_Header_Straight_2x20" H 3550 2150 60  0001 C CNN
-F 3 "" H 3550 2150 60  0000 C CNN
-	1    3550 2150
-	1    0    0    -1
-$EndComp
-$Comp
-L power:GND #PWR0102
-U 1 1 604AF549
-P 3200 4150
-F 0 "#PWR0102" H 3200 3900 50  0001 C CNN
-F 1 "GND" H 3205 3977 50  0000 C CNN
-F 2 "" H 3200 4150 50  0001 C CNN
-F 3 "" H 3200 4150 50  0001 C CNN
-	1    3200 4150
-	1    0    0    -1
-$EndComp
-$Comp
-L power:GND #PWR0103
-U 1 1 604B0835
-P 5400 4150
-F 0 "#PWR0103" H 5400 3900 50  0001 C CNN
-F 1 "GND" H 5405 3977 50  0000 C CNN
-F 2 "" H 5400 4150 50  0001 C CNN
-F 3 "" H 5400 4150 50  0001 C CNN
-	1    5400 4150
-	1    0    0    -1
-$EndComp
-Wire Wire Line
-	5250 2350 5400 2350
-Wire Wire Line
-	5400 2350 5400 2750
-Wire Wire Line
-	5250 2750 5400 2750
-Connection ~ 5400 2750
-Wire Wire Line
-	5400 2750 5400 3050
-Wire Wire Line
-	5250 3050 5400 3050
-Connection ~ 5400 3050
-Wire Wire Line
-	5400 3050 5400 3550
-Wire Wire Line
-	5250 3550 5400 3550
-Connection ~ 5400 3550
-Wire Wire Line
-	5400 3550 5400 3750
-Wire Wire Line
-	5250 3750 5400 3750
-Connection ~ 5400 3750
-Wire Wire Line
-	5400 3750 5400 4150
-Wire Wire Line
-	3200 4150 3200 4050
-Wire Wire Line
-	3200 2550 3350 2550
-Wire Wire Line
-	3350 3350 3200 3350
-Connection ~ 3200 3350
-Wire Wire Line
-	3200 3350 3200 2550
-Wire Wire Line
-	3350 4050 3200 4050
-Connection ~ 3200 4050
-Wire Wire Line
-	3200 4050 3200 3350
-$Comp
-L Device:D_Schottky D26
-U 1 1 605A89CC
-P 9500 2350
-F 0 "D26" H 9500 2567 50  0000 C CNN
-F 1 "D_Schottky" H 9500 2476 50  0000 C CNN
-F 2 "Diode_SMD:D_SOD-128" H 9500 2350 50  0001 C CNN
-F 3 "~" H 9500 2350 50  0001 C CNN
-	1    9500 2350
-	1    0    0    -1
-$EndComp
-$Comp
-L power:+5V #PWR0106
-U 1 1 605AA90B
-P 9650 2350
-F 0 "#PWR0106" H 9650 2200 50  0001 C CNN
-F 1 "+5V" V 9650 2450 50  0000 L CNN
-F 2 "" H 9650 2350 50  0001 C CNN
-F 3 "" H 9650 2350 50  0001 C CNN
-	1    9650 2350
-	0    1    1    0
-$EndComp
-$Comp
-L power:+5V #PWR0107
-U 1 1 605AC150
-P 5250 2050
-F 0 "#PWR0107" H 5250 1900 50  0001 C CNN
-F 1 "+5V" H 5265 2223 50  0000 C CNN
-F 2 "" H 5250 2050 50  0001 C CNN
-F 3 "" H 5250 2050 50  0001 C CNN
-	1    5250 2050
-	1    0    0    -1
-$EndComp
-Wire Wire Line
-	5250 2250 5250 2150
-Wire Wire Line
-	5250 2150 5250 2050
-Connection ~ 5250 2150
-$Comp
 L power:+3V3 #PWR0115
 U 1 1 608B771D
@@
 Wire Wire Line
 	7050 2350 6550 2350
-Text Label 5750 2450 0    50   ~ 0
-PI_TX
-Text Label 5750 2550 0    50   ~ 0
-PI_RX
 $Comp
 L teensy:Teensy4.1 U10
@@
 Wire Wire Line
 	7050 3950 6700 3950
-Wire Wire Line
-	5250 2450 7050 2450
-Wire Wire Line
-	5250 2550 7050 2550
 Text HLabel 9900 4550 2    50   Output ~ 0
 CS0
@@
 Wire Wire Line
 	9650 4550 9900 4550
-Wire Wire Line
-	3350 3250 3050 3250
-Wire Wire Line
-	3350 3150 3050 3150
-Wire Wire Line
-	3350 3050 3050 3050
 Text HLabel 9950 4450 2    50   Output ~ 0
 CS2
@@
 Wire Wire Line
 	9950 4350 9650 4350
-Text Label 5550 2950 0    50   ~ 0
-SWDIO
-Text Label 5550 3150 0    50   ~ 0
-SCLK
-Wire Wire Line
-	5250 2950 5550 2950
-Wire Wire Line
-	5250 3150 5550 3150
 Text HLabel 6500 3550 0    50   Input ~ 0
 SPI_MOSI
@@
 F 2 "Resistor_SMD:R_0603_1608Metric_Pad0.98x0.95mm_HandSolder" H 9350 4650 50  0001 C CNN
 F 3 "~" H 9350 4650 50  0001 C CNN
+F 4 "C105588" H 9350 4650 50  0001 C CNN "LCSC"
 	1    9350 4650
 	0    -1   -1   0
@@
 F 2 "Resistor_SMD:R_0603_1608Metric_Pad0.98x0.95mm_HandSolder" H 6950 3550 50  0001 C CNN
 F 3 "~" H 6950 3550 50  0001 C CNN
+F 4 "C105588" H 6950 3550 50  0001 C CNN "LCSC"
 	1    6950 3550
 	0    -1   -1   0
@@
 F 2 "Resistor_SMD:R_0603_1608Metric_Pad0.98x0.95mm_HandSolder" H 9350 3650 50  0001 C CNN
 F 3 "~" H 9350 3650 50  0001 C CNN
+F 4 "C105588" H 9350 3650 50  0001 C CNN "LCSC"
 	1    9350 3650
 	0    -1   -1   0
@@
 F 2 "Resistor_SMD:R_Array_Concave_4x0603" V 9725 4350 50  0001 C CNN
 F 3 "~" H 9450 4350 50  0001 C CNN
+F 4 "742C083101JPCT-ND" V 9450 4350 50  0001 C CNN "Digi-Key_PN"
+F 5 "C79203" V 9450 4350 50  0001 C CNN "LCSC"
 	1    9450 4350
 	0    1    -1   0
@@
 Wire Wire Line
 	9450 4650 9700 4650
+$Comp
+L power:+5V #PWR0106
+U 1 1 605AA90B
+P 9650 2350
+F 0 "#PWR0106" H 9650 2200 50  0001 C CNN
+F 1 "+5V" V 9650 2450 50  0000 L CNN
+F 2 "" H 9650 2350 50  0001 C CNN
+F 3 "" H 9650 2350 50  0001 C CNN
+	1    9650 2350
+	0    1    1    0
+$EndComp
+$Comp
+L Device:D_Schottky D26
+U 1 1 605A89CC
+P 9500 2350
+F 0 "D26" H 9500 2567 50  0000 C CNN
+F 1 "D_Schottky" H 9500 2476 50  0000 C CNN
+F 2 "Diode_SMD:D_SOD-128" H 9500 2350 50  0001 C CNN
+F 3 "~" H 9500 2350 50  0001 C CNN
+F 4 "1727-7810-1-ND" H 9500 2350 50  0001 C CNN "Digi-Key_PN"
+F 5 "C456127" H 9500 2350 50  0001 C CNN "LCSC"
+	1    9500 2350
+	1    0    0    -1
+$EndComp
 $EndSCHEMATC

Commit message: pre delete thru hole
Parts:
- added J35: MICROMOD-2222-C, SparkFun-MicroMod:M.2-CONNECTOR-E, symbol MicroMod_Processor_Board:MICROMOD-2222-C
- added J36, J37: Conn_01x02_Male, Connector_PinHeader_2.54mm:PinHeader_1x02_P2.54mm_Vertical, symbol Connector:Conn_01x02_Male
- added R13, R14, R15: 100, Resistor_SMD:R_0603_1608Metric_Pad0.98x0.95mm_HandSolder, symbol Device:R_Small_US
- added RN4: R_100_4, Resistor_SMD:R_Array_Concave_4x0603, symbol Device:R_Pack04
Connections:
- net +5V: now also J35.9 (USB_VIN)
- net A_DIR: now also J35.69 (G7/BUS7)
- net A_ENABLE: now also J35.68 (SDIO_DATA2)
- net A_ENCA: now also J35.58 (AUD_MCLK)
- net A_ENCB: now also J35.14 (I2C_SCL)
- net A_STEP: now also J35.54 (AUD_IN/CAM_PCLK)
- net B_DIR: now also J35.8 (G11)
- net B_ENABLE: now also J35.42 (G1/BUS1)
- net B_ENCA: now also J35.4 (3.3V_EN)
- net B_ENCB: now also J35.41 (CAN-RX)
- net B_STEP: now also J35.67 (G8)
- net CS0: now also RN4.8 (R1.2)
- net CS1: now also R15.2
- net CS2: now also RN4.7 (R2.2)
- net CS3: now also RN4.6 (R3.2)
- net CS4: now also RN4.5 (R4.2)
- net GND: now also J35.1 (GND), J35.33 (GND), J35.36 (GND), J35.39 (GND), J35.45 (GND), J35.7 (GND), J35.75 (GND), J36.2 (Pin_2), J37.2 (Pin_2)
- net SCL: now also J35.53 (I2C_SCL1)
- net SDA: now also J35.51 (I2C_SDA1)
- net SPI_CLK: now also R13.2
- net SPI_MISO: now also J35.61 (SPI_SDI)
- net SPI_MOSI: now also R14.1
- net X_DIR: now also J35.32 (PWM0)
- net X_EN: now also J35.55 (SPI_~CS~)
- net X_LIMIT: now also J35.52 (AUD_LRCLK)
- net X_STEP: now also J35.47 (PWM1)
- net Y_DIR: now also J35.18 (D1/CAM_TRIG)
- net Y_ENABLE: now also J35.40 (G0/BUS0)
- net Y_STEP: now also J35.10 (D0)
- net Z_DIR: now also J35.56 (AUD_OUT/CAM_MCLK)
- net Z_ENABLE: now also J35.70 (SPI_~CS1~/SDIO_DATA3)
- net Z_LIMIT: now also J35.49 (BATT_VIN/3)
- net Z_STEP: now also J35.71 (G6/BUS6)
- new net: J35.11 (~BOOT~), J37.1 (Pin_1)
- new net: J35.57 (SPI_SCK), R13.1
- new net: J35.59 (SPI_SDO), R14.2
- new net: J35.6 (~RESET~), J36.1 (Pin_1)
- new net: J35.60 (SPI_SCK1/SDIO_CLK), RN4.3 (R3.1)
- new net: J35.62 (SPI_SDO1/SDIO_CMD), RN4.4 (R4.1)
- new net: J35.63 (G10/ADC_D+/CAM_VSYNC), R15.1
- new net: J35.64 (SPI_SDI1/SDIO_DATA0), RN4.2 (R2.1)
- new net: J35.66 (SDIO_DATA1), RN4.1 (R1.1)
- new net +3.3VA: J35.2 (3.3V), J35.74 (3.3V)
- new net USB_TEENSY_N: J35.5 (USB_D-)
- new net USB_TEENSY_P: J35.3 (USB_D+)

Commit message: trying new stuff
Parts:
- removed D26: D_Schottky, Diode_SMD:D_SOD-128, symbol Device:D_Schottky
- removed R5, R6, R7: 100, Resistor_SMD:R_0603_1608Metric_Pad0.98x0.95mm_HandSolder, symbol Device:R_Small_US
- removed RN3: R_100_4, Resistor_SMD:R_Array_Concave_4x0603, symbol Device:R_Pack04
- removed U10: Teensy4.1, teensy:Teensy41, symbol teensy:Teensy4.1
Connections:
- net Y_LIMIT: now also J35.50 (AUD_BCLK)
Other:
- moved on the sheet: J35, J36, J37, R13, R14, R15, RN4

Commit message: bunches of changes
Changed lines of the file:
@@
 Wire Wire Line
 	4800 4200 4950 4200
+$Comp
+L power:+3.3V #PWR0101
+U 1 1 616D7C7A
+P 4850 1800
+F 0 "#PWR0101" H 4850 1650 50  0001 C CNN
+F 1 "+3.3V" H 4865 1973 50  0000 C CNN
+F 2 "" H 4850 1800 50  0001 C CNN
+F 3 "" H 4850 1800 50  0001 C CNN
+	1    4850 1800
+	1    0    0    -1
+$EndComp
+Wire Wire Line
+	4850 1800 4950 1800
+Connection ~ 4950 1800
 $EndSCHEMATC
