File: electrical/stepper_multi_axis/Stepper_Driver_X.sch (KiCad schematic (older format))
At the start: 11 parts, among them J1 Conn_01x04_Male, J4 Conn_01x03_Male, U2 TMC5160_SILENTSTEPSTICK, U3 LTV-817

Commit message: shipped things
Parts:
- C1: Digi-Key_PN (none) -> PCE4976CT-ND
- C8: LCSC (none) -> C83054
- D27: LCSC (none) -> C434419
- J1: Digi-Key_PN (none) -> WM22669-ND
- J4: Digi-Key_PN (none) -> WM22668-ND
- R26, R27, R28: LCSC (none) -> C105588
- U2: Digi-Key_PN (none) -> 1460-TMC5160SILENTSTEPSTICK-ND
- U3: footprint Package_DIP:DIP-4_W7.62mm_SMDSocket_SmallPads -> Package_DIP:DIP-4_W8.89mm_SMDSocket_LongPads; Digi-Key_PN (none) -> 160-1893-1-ND; JLCPCB C106900 -> (none); LCSC (none) -> C106900
Changed lines of the file:
@@
 $Descr A4 11693 8268
 encoding utf-8
-Sheet 6 8
+Sheet 6 10
 Title ""
 Date ""
@@
 F 6 "Trinamic" H 5050 3500 50  0001 L BNN "MANUFACTURER"
 F 7 "Manufacturer Recommendations" H 5050 3500 50  0001 L BNN "STANDARD"
+F 8 "1460-TMC5160SILENTSTEPSTICK-ND" H 5050 3500 50  0001 C CNN "Digi-Key_PN"
 	1    5050 3500
 	1    0    0    -1
@@
 F 2 "Capacitor_SMD:CP_Elec_8x6.7" H 6650 2750 50  0001 C CNN
 F 3 "~" H 6650 2750 50  0001 C CNN
+F 4 "PCE4976CT-ND" H 6650 2750 50  0001 C CNN "Digi-Key_PN"
 	1    6650 2750
 	1    0    0    -1
@@
 F 0 "U3" H 4950 2075 50  0000 C CNN
 F 1 "LTV-817" H 4950 1984 50  0000 C CNN
-F 2 "Package_DIP:DIP-4_W7.62mm_SMDSocket_SmallPads" H 4750 1550 50  0001 L CIN
+F 2 "Package_DIP:DIP-4_W8.89mm_SMDSocket_LongPads" H 4750 1550 50  0001 L CIN
 F 3 "http://www.us.liteon.com/downloads/LTV-817-827-847.PDF" H 4950 1650 50  0001 L CNN
-F 4 "C106900" H 4950 1750 50  0001 C CNN "JLCPCB"
+F 4 "C106900" H 4950 1750 50  0001 C CNN "LCSC"
+F 5 "160-1893-1-ND" H 4950 1750 50  0001 C CNN "Digi-Key_PN"
 	1    4950 1750
 	-1   0    0    -1
@@
 F 2 "Resistor_SMD:R_0603_1608Metric_Pad0.98x0.95mm_HandSolder" H 5250 1400 50  0001 C CNN
 F 3 "~" H 5250 1400 50  0001 C CNN
+F 4 "C105588" H 5250 1400 50  0001 C CNN "LCSC"
 	1    5250 1400
 	1    0    0    -1
@@
 F 2 "LED_SMD:LED_0603_1608Metric_Pad1.05x0.95mm_HandSolder" H 5550 1650 50  0001 C CNN
 F 3 "~" H 5550 1650 50  0001 C CNN
+F 4 "C434419" H 5550 1650 50  0001 C CNN "LCSC"
 	1    5550 1650
 	0    -1   -1   0
@@
 F 2 "Resistor_SMD:R_0603_1608Metric_Pad0.98x0.95mm_HandSolder" H 5550 1400 50  0001 C CNN
 F 3 "~" H 5550 1400 50  0001 C CNN
+F 4 "C105588" H 5550 1400 50  0001 C CNN "LCSC"
 	1    5550 1400
 	1    0    0    -1
@@
 F 2 "Resistor_SMD:R_0603_1608Metric_Pad0.98x0.95mm_HandSolder" H 4650 2050 50  0001 C CNN
 F 3 "~" H 4650 2050 50  0001 C CNN
+F 4 "C105588" H 4650 2050 50  0001 C CNN "LCSC"
 	1    4650 2050
 	1    0    0    -1
@@
 F 2 "Capacitor_SMD:C_0603_1608Metric_Pad1.08x0.95mm_HandSolder" H 4500 2050 50  0001 C CNN
 F 3 "~" H 4500 2050 50  0001 C CNN
+F 4 "C83054" H 4500 2050 50  0001 C CNN "LCSC"
 	1    4500 2050
 	-1   0    0    1
@@
 F 2 "sl_connector:1719740104" H 6350 3500 50  0001 C CNN
 F 3 "~" H 6350 3500 50  0001 C CNN
+F 4 "WM22669-ND" H 6350 3500 50  0001 C CNN "Digi-Key_PN"
 	1    6350 3500
 	-1   0    0    -1
@@
 F 2 "sl_connector:1719740103" H 6250 1750 50  0001 C CNN
 F 3 "~" H 6250 1750 50  0001 C CNN
+F 4 "WM22668-ND" H 6250 1750 50  0001 C CNN "Digi-Key_PN"
 	1    6250 1750
 	-1   0    0    -1

Commit message: bunches of changes
Changed lines of the file:
@@
 $Descr A4 11693 8268
 encoding utf-8
-Sheet 6 10
+Sheet 5 10
 Title ""
 Date ""
@@
 AR Path="/608FE26D/60870DCB" Ref="#PWR0123"  Part="1"
 AR Path="/608FE277/60870DCB" Ref="#PWR0130"  Part="1"
-F 0 "#PWR0108" H 5750 4150 50  0001 C CNN
+F 0 "#PWR0123" H 5750 4150 50  0001 C CNN
 F 1 "GND" H 5755 4227 50  0000 C CNN
 F 2 "" H 5750 4400 50  0001 C CNN
@@
 AR Path="/608FE26D/608718E9" Ref="#PWR0124"  Part="1"
 AR Path="/608FE277/608718E9" Ref="#PWR0131"  Part="1"
-F 0 "#PWR0109" H 6050 2500 50  0001 C CNN
+F 0 "#PWR0124" H 6050 2500 50  0001 C CNN
 F 1 "VBUS" H 6065 2823 50  0000 C CNN
 F 2 "" H 6050 2650 50  0001 C CNN
@@
 AR Path="/608FE26D/60872ABF" Ref="#PWR0125"  Part="1"
 AR Path="/608FE277/60872ABF" Ref="#PWR0132"  Part="1"
-F 0 "#PWR0110" H 5850 2600 50  0001 C CNN
+F 0 "#PWR0125" H 5850 2600 50  0001 C CNN
 F 1 "+3V3" H 5865 2923 50  0000 C CNN
 F 2 "" H 5850 2750 50  0001 C CNN
@@
 AR Path="/608FE26D/6086E8C9" Ref="U7"  Part="1"
 AR Path="/608FE277/6086E8C9" Ref="U9"  Part="1"
-F 0 "U2" H 5050 4367 50  0000 C CNN
+F 0 "U7" H 5050 4367 50  0000 C CNN
 F 1 "TMC5160_SILENTSTEPSTICK" H 5050 4276 50  0000 C CNN
 F 2 "Trinamic:MODULE_TMC_SILENTSTEPSTICK" H 5050 3500 50  0001 L BNN
@@
 AR Path="/608FE26D/60876F12" Ref="C3"  Part="1"
 AR Path="/608FE277/60876F12" Ref="C4"  Part="1"
-F 0 "C1" H 6765 2796 50  0000 L CNN
+F 0 "C3" H 6765 2796 50  0000 L CNN
 F 1 "10uF" H 6765 2705 50  0000 L CNN
 F 2 "Capacitor_SMD:CP_Elec_8x6.7" H 6650 2750 50  0001 C CNN
@@
 AR Path="/608FE26D/608785AC" Ref="#PWR0126"  Part="1"
 AR Path="/608FE277/608785AC" Ref="#PWR0133"  Part="1"
-F 0 "#PWR0111" H 6650 2650 50  0001 C CNN
+F 0 "#PWR0126" H 6650 2650 50  0001 C CNN
 F 1 "GND" H 6655 2727 50  0000 C CNN
 F 2 "" H 6650 2900 50  0001 C CNN
@@
 AR Path="/608FE26D/60878CAB" Ref="#PWR0127"  Part="1"
 AR Path="/608FE277/60878CAB" Ref="#PWR0134"  Part="1"
-F 0 "#PWR0112" H 6650 2450 50  0001 C CNN
+F 0 "#PWR0127" H 6650 2450 50  0001 C CNN
 F 1 "VBUS" H 6665 2773 50  0000 C CNN
 F 2 "" H 6650 2600 50  0001 C CNN
@@
 AR Path="/608FE26D/608834B7" Ref="U6"  Part="1"
 AR Path="/608FE277/608834B7" Ref="U8"  Part="1"
-F 0 "U3" H 4950 2075 50  0000 C CNN
+F 0 "U6" H 4950 2075 50  0000 C CNN
 F 1 "LTV-817" H 4950 1984 50  0000 C CNN
 F 2 "Package_DIP:DIP-4_W8.89mm_SMDSocket_LongPads" H 4750 1550 50  0001 L CIN
@@
 AR Path="/608FE26D/60889A9D" Ref="#PWR0128"  Part="1"
 AR Path="/608FE277/60889A9D" Ref="#PWR0135"  Part="1"
-F 0 "#PWR0113" H 4650 1000 50  0001 C CNN
+F 0 "#PWR0128" H 4650 1000 50  0001 C CNN
 F 1 "+3V3" H 4665 1323 50  0000 C CNN
 F 2 "" H 4650 1150 50  0001 C CNN
@@
 AR Path="/608FE26D/6088A387" Ref="#PWR0129"  Part="1"
 AR Path="/608FE277/6088A387" Ref="#PWR0136"  Part="1"
-F 0 "#PWR0114" H 4650 2050 50  0001 C CNN
+F 0 "#PWR0129" H 4650 2050 50  0001 C CNN
 F 1 "GND" H 4655 2127 50  0000 C CNN
 F 2 "" H 4650 2300 50  0001 C CNN
@@
 AR Path="/608FE26D/60890195" Ref="R33"  Part="1"
 AR Path="/608FE277/60890195" Ref="R36"  Part="1"
-F 0 "R27" H 5318 1446 50  0000 L CNN
+F 0 "R33" H 5318 1446 50  0000 L CNN
 F 1 "100" H 5318 1355 50  0000 L CNN
 F 2 "Resistor_SMD:R_0603_1608Metric_Pad0.98x0.95mm_HandSolder" H 5250 1400 50  0001 C CNN
@@
 AR Path="/608FE26D/608A1732" Ref="D29"  Part="1"
 AR Path="/608FE277/608A1732" Ref="D30"  Part="1"
-F 0 "D27" H 5543 1867 50  0000 C CNN
+F 0 "D29" H 5543 1867 50  0000 C CNN
 F 1 "LED" H 5543 1776 50  0000 C CNN
 F 2 "LED_SMD:LED_0603_1608Metric_Pad1.05x0.95mm_HandSolder" H 5550 1650 50  0001 C CNN
@@
 AR Path="/608FE26D/608A77D0" Ref="R34"  Part="1"
 AR Path="/608FE277/608A77D0" Ref="R37"  Part="1"
-F 0 "R28" H 5618 1446 50  0000 L CNN
+F 0 "R34" H 5618 1446 50  0000 L CNN
 F 1 "100" H 5618 1355 50  0000 L CNN
 F 2 "Resistor_SMD:R_0603_1608Metric_Pad0.98x0.95mm_HandSolder" H 5550 1400 50  0001 C CNN
@@
 AR Path="/608FE26D/60888114" Ref="R32"  Part="1"
 AR Path="/608FE277/60888114" Ref="R35"  Part="1"
-F 0 "R26" H 4718 2096 50  0000 L CNN
+F 0 "R32" H 4718 2096 50  0000 L CNN
 F 1 "100" H 4718 2005 50  0000 L CNN
 F 2 "Resistor_SMD:R_0603_1608Metric_Pad0.98x0.95mm_HandSolder" H 4650 2050 50  0001 C CNN
@@
 AR Path="/608DFF6C/60A5FD43" Ref="C6"  Part="1"
 AR Path="/608FE26D/60A5FD43" Ref="C7"  Part="1"
-F 0 "C5" H 4800 2000 50  0000 R CNN
+F 0 "C7" H 4800 2000 50  0000 R CNN
 F 1 "100nF" H 4800 2100 50  0000 R CNN
 F 2 "Capacitor_SMD:C_0603_1608Metric_Pad1.08x0.95mm_HandSolder" H 4500 2050 50  0001 C CNN
@@
 AR Path="/608FE26D/60F78CCC" Ref="J7"  Part="1"
 AR Path="/608FE277/60F78CCC" Ref="J9"  Part="1"
-F 0 "J1" H 6322 3474 50  0000 R CNN
+F 0 "J7" H 6322 3474 50  0000 R CNN
 F 1 "Conn_01x04_Male" H 6322 3383 50  0000 R CNN
 F 2 "sl_connector:1719740104" H 6350 3500 50  0001 C CNN
@@
 AR Path="/608FE26D/60F911B2" Ref="J6"  Part="1"
 AR Path="/608FE277/60F911B2" Ref="J8"  Part="1"
-F 0 "J3" H 6222 1774 50  0000 R CNN
+F 0 "J6" H 6222 1774 50  0000 R CNN
 F 1 "Conn_01x03_Male" H 6222 1683 50  0000 R CNN
 F 2 "sl_connector:1719740103" H 6250 1750 50  0001 C CNN
@@
 AR Path="/608FE26D/610652DE" Ref="R3"  Part="1"
 AR Path="/608FE277/610652DE" Ref="R4"  Part="1"
-F 0 "R1" H 4318 3846 50  0000 L CNN
+F 0 "R3" H 4318 3846 50  0000 L CNN
 F 1 "100" H 4318 3755 50  0000 L CNN
 F 2 "Resistor_SMD:R_0603_1608Metric_Pad0.98x0.95mm_HandSolder" H 4250 3800 50  0001 C CNN
